File: kudox-game/rev2/kudox_game.kicad_pcb (KiCad board)
At the start: 2 copper layers, 145.7 x 130.4 mm, 68 parts, among them K0 KEYSW, K1 KEYSW, K11 KEYSW, K12 KEYSW, K13 KEYSW, K14 KEYSW, K15 KEYSW, K2 KEYSW, K20 KEYSW, K21 KEYSW, K22 KEYSW, K23 KEYSW, K24 KEYSW, K25 KEYSW, K26 KEYSW, K3 KEYSW, K30 KEYSW, K31 KEYSW, K34 KEYSW, K35 KEYSW, K36 KEYSW, K4 KEYSW, K40 KEYSW, K45 KEYSW, K46 KEYSW, K5 KEYSW, U1 ProMicro

Commit message: rgb stuff
Parts:
- removed G*** (x2): LOGO, kudox_game_footprints:qmk-badge-pad
- removed G*** (x2): kudox_github, kudox_game_footprints:kudox_github
- removed G*** (x2): LOGO, kudox_game_footprints:kudox_game_logo_pad
- removed G*** (x2): LOGO, kudox_game_footprints:version
- removed HOLE_M3 (x5): VAL**, keyboard_parts:HOLE_M3
- removed RGB_STRIP1: RGB_STRIP, kudox_game_footprints:Pin_Header_Straight_1x03_Pitch2.54mm
- removed RST_SW1: SW_PUSH, kudox_game_footprints:SW_PUSH_6mm_h4.3mm
- added C1: 22pF, 3x6_components:C_0805_2012Metric_Pad1.18x1.45mm_HandSolder, F.Cu at (49.5, 52.5)
- added C10: 0.1uF, 3x6_components:C_0603_1608Metric_Pad1.08x0.95mm_HandSolder, B.Cu at (138.2, 90.7)
- added C11: 0.1uF, 3x6_components:C_0603_1608Metric_Pad1.08x0.95mm_HandSolder, B.Cu at (57.5, 38.9)
- added C12: 0.1uF, 3x6_components:C_0603_1608Metric_Pad1.08x0.95mm_HandSolder, B.Cu at (174.1, 76.3)
- added C13: 0.1uF, 3x6_components:C_0603_1608Metric_Pad1.08x0.95mm_HandSolder, B.Cu at (161.6, 131.6)
- added C14: 0.1uF, 3x6_components:C_0603_1608Metric_Pad1.08x0.95mm_HandSolder, B.Cu at (154.8, 77.3)
- added C15: 0.1uF, 3x6_components:C_0603_1608Metric_Pad1.08x0.95mm_HandSolder, B.Cu at (158.7, 52.2)
- added C16: 0.1uF, 3x6_components:C_0603_1608Metric_Pad1.08x0.95mm_HandSolder, B.Cu at (77.8, 90.8)
- added C17: 0.1uF, 3x6_components:C_0603_1608Metric_Pad1.08x0.95mm_HandSolder, B.Cu at (57.0, 76.4)
- added C18: 0.1uF, 3x6_components:C_0603_1608Metric_Pad1.08x0.95mm_HandSolder, B.Cu at (160.6, 38.1)
- added C19: 0.1uF, 3x6_components:C_0603_1608Metric_Pad1.08x0.95mm_HandSolder, B.Cu at (86.8, 37.5)
- added C2: 22pF, 3x6_components:C_0805_2012Metric_Pad1.18x1.45mm_HandSolder, F.Cu at (58.1, 52.4)
- added C20: 0.1uF, 3x6_components:C_0603_1608Metric_Pad1.08x0.95mm_HandSolder, B.Cu at (55.8, 89.8)
- added C21: 0.1uF, 3x6_components:C_0603_1608Metric_Pad1.08x0.95mm_HandSolder, B.Cu at (62.6, 113.6)
- added C22: 0.1uF, 3x6_components:C_0603_1608Metric_Pad1.08x0.95mm_HandSolder, B.Cu at (132.7, 77.3)
- added C23: 0.1uF, 3x6_components:C_0603_1608Metric_Pad1.08x0.95mm_HandSolder, B.Cu at (75.5, 77.4)
- added C24: 0.1uF, 3x6_components:C_0603_1608Metric_Pad1.08x0.95mm_HandSolder, B.Cu at (105.8, 37.5)
- added C25: 0.1uF, 3x6_components:C_0603_1608Metric_Pad1.08x0.95mm_HandSolder, B.Cu at (158.1, 89.8)
- added C26: 0.1uF, 3x6_components:C_0603_1608Metric_Pad1.08x0.95mm_HandSolder, B.Cu at (182.1, 146.1)
- added C27: 0.1uF, 3x6_components:C_0603_1608Metric_Pad1.08x0.95mm_HandSolder, B.Cu at (113.6, 77.4)
- added C28: 0.1uF, 3x6_components:C_0603_1608Metric_Pad1.08x0.95mm_HandSolder, B.Cu at (137.9, 52.9)
- added C29: 0.1uF, 3x6_components:C_0603_1608Metric_Pad1.08x0.95mm_HandSolder, B.Cu at (119.2, 90.7)
- added C3: 10uF, 3x6_components:C_0805_2012Metric_Pad1.18x1.45mm_HandSolder, F.Cu at (62.0, 60.6)
- added C30: 0.1uF, 3x6_components:C_0603_1608Metric_Pad1.08x0.95mm_HandSolder, B.Cu at (83.6, 52.1)
- added C31: 0.1uF, 3x6_components:C_0603_1608Metric_Pad1.08x0.95mm_HandSolder, B.Cu at (143.7, 37.6)
- added C32: 0.1uF, 3x6_components:C_0603_1608Metric_Pad1.08x0.95mm_HandSolder, B.Cu at (119.0, 52.9)
- added C33: 0.1uF, 3x6_components:C_0603_1608Metric_Pad1.08x0.95mm_HandSolder, B.Cu at (125.0, 37.6)
- added C34: 0.1uF, 3x6_components:C_0603_1608Metric_Pad1.08x0.95mm_HandSolder, B.Cu at (99.8, 53.0)
- added C35: 0.1uF, 3x6_components:C_0603_1608Metric_Pad1.08x0.95mm_HandSolder, B.Cu at (94.6, 77.4)
- added C4: 1uF, 3x6_components:C_0805_2012Metric_Pad1.18x1.45mm_HandSolder, F.Cu at (63.0, 66.1)
- added C5: 1uF, 3x6_components:C_0805_2012Metric_Pad1.18x1.45mm_HandSolder, F.Cu at (62.0, 62.6)
- added C6: 0.1uF, 3x6_components:C_0805_2012Metric_Pad1.18x1.45mm_HandSolder, F.Cu at (61.0, 56.3)
- added C7: 0.1uF, 3x6_components:C_0805_2012Metric_Pad1.18x1.45mm_HandSolder, F.Cu at (63.0, 56.3)
- added C8: 0.1uF, 3x6_components:C_0805_2012Metric_Pad1.18x1.45mm_HandSolder, F.Cu at (46.7, 54.0)
- added C9: 0.1uF, 3x6_components:C_0805_2012Metric_Pad1.18x1.45mm_HandSolder, F.Cu at (44.7, 54.0)
- added F1: 500mA, 3x6_components:Fuse_1206_3216Metric_Pad1.42x1.75mm_HandSolder, F.Cu at (63.0, 50.4)
- added H1: ThroughHole, kudox_game_footprints:HOLE_M3, F.Cu at (67.4, 41.7)
- added H2: ThroughHole, kudox_game_footprints:HOLE_M3, F.Cu at (173.1, 40.8)
- added H3: ThroughHole, kudox_game_footprints:HOLE_M3, F.Cu at (177.6, 111.8)
- added H4: ThroughHole, kudox_game_footprints:HOLE_M3, F.Cu at (102.8, 117.8)
- added H5: ThroughHole, kudox_game_footprints:HOLE_M3, F.Cu at (177.3, 156.1)
- added LED0: SK6812MINI-E, 3x6_components:LED_MX_SK6812MINI-E, F.Cu at (53.4, 40.9)
- added LED1: SK6812MINI-E, 3x6_components:LED_MX_SK6812MINI-E, F.Cu at (81.4, 40.9)
- added LED11: SK6812MINI-E, 3x6_components:LED_MX_SK6812MINI-E_REV, F.Cu at (86.2, 59.9)
- added LED12: SK6812MINI-E, 3x6_components:LED_MX_SK6812MINI-E_REV, F.Cu at (105.2, 59.9)
- added LED13: SK6812MINI-E, 3x6_components:LED_MX_SK6812MINI-E_REV, F.Cu at (124.3, 59.9)
- added LED14: SK6812MINI-E, 3x6_components:LED_MX_SK6812MINI-E_REV, F.Cu at (143.3, 59.9)
- added LED15: SK6812MINI-E, 3x6_components:LED_MX_SK6812MINI-E_REV, F.Cu at (162.4, 59.9)
- added LED2: SK6812MINI-E, 3x6_components:LED_MX_SK6812MINI-E, F.Cu at (100.5, 40.9)
- added LED20: SK6812MINI-E, 3x6_components:LED_MX_SK6812MINI-E, F.Cu at (53.4, 78.9)
- added LED21: SK6812MINI-E, 3x6_components:LED_MX_SK6812MINI-E, F.Cu at (72.4, 78.9)
- added LED22: SK6812MINI-E, 3x6_components:LED_MX_SK6812MINI-E, F.Cu at (91.5, 78.9)
- added LED23: SK6812MINI-E, 3x6_components:LED_MX_SK6812MINI-E, F.Cu at (110.5, 78.9)
- added LED24: SK6812MINI-E, 3x6_components:LED_MX_SK6812MINI-E, F.Cu at (129.6, 78.9)
- added LED25: SK6812MINI-E, 3x6_components:LED_MX_SK6812MINI-E, F.Cu at (151.7, 78.9)
- added LED26: SK6812MINI-E, 3x6_components:LED_MX_SK6812MINI-E, F.Cu at (170.8, 78.9)
- added LED3: SK6812MINI-E, 3x6_components:LED_MX_SK6812MINI-E, F.Cu at (119.5, 40.9)
- added LED30: SK6812MINI-E, 3x6_components:LED_MX_SK6812MINI-E_REV, F.Cu at (58.1, 98.0)
- added LED31: SK6812MINI-E, 3x6_components:LED_MX_SK6812MINI-E_REV, F.Cu at (82.6, 98.0)
- added LED34: SK6812MINI-E, 3x6_components:LED_MX_SK6812MINI-E_REV, F.Cu at (124.0, 98.0)
- added LED35: SK6812MINI-E, 3x6_components:LED_MX_SK6812MINI-E_REV, F.Cu at (143.1, 98.0)
- added LED36: SK6812MINI-E, 3x6_components:LED_MX_SK6812MINI-E_REV, F.Cu at (162.1, 98.0)
- added LED4: SK6812MINI-E, 3x6_components:LED_MX_SK6812MINI-E, F.Cu at (138.6, 40.9)
- added LED40: SK6812MINI-E, 3x6_components:LED_MX_SK6812MINI-E, F.Cu at (58.1, 117.0)
- added LED45: SK6812MINI-E, 3x6_components:LED_MX_SK6812MINI-E, F.Cu at (158.1, 126.6)
- added LED46: SK6812MINI-E, 3x6_components:LED_MX_SK6812MINI-E, F.Cu at (176.9, 140.5)
- added LED5: SK6812MINI-E, 3x6_components:LED_MX_SK6812MINI-E, F.Cu at (157.6, 40.9)
- added LOGO1: arisutea_logo, 3x6_graphics:warning_sign_3.6x3.2mm, F.Cu at (306.4, 155.8)
- added LOGO2: arisutea_logo, 3x6_graphics:warning_sign_3.6x3.2mm, F.Cu at (308.4, 160.7)
- added LOGO3: OSHW Logo, 3x6_graphics:osh-logo, F.Cu at (307.0, 130.5)
- added LOGO4: OSHW Logo, 3x6_graphics:osh-logo, F.Cu at (307.1, 121.2)
- added LOGO5: QMK_Logo_Light, 3x6_graphics:QMK_Logo_Light, F.Cu at (308.0, 149.9)
- added LOGO6: QMK_Logo_Light, 3x6_graphics:QMK_Logo_Light, F.Cu at (306.8, 142.6)
- added R1: 22, 3x6_components:R_0805_2012Metric_Pad1.20x1.40mm_HandSolder, F.Cu at (68.2, 55.2)
- added R2: 10K, 3x6_components:R_0805_2012Metric_Pad1.20x1.40mm_HandSolder, F.Cu at (63.1, 68.2)
- added R3: 5k1, 3x6_components:R_0805_2012Metric_Pad1.20x1.40mm_HandSolder, F.Cu at (77.2, 32.2)
- added R4: 5k1, 3x6_components:R_0805_2012Metric_Pad1.20x1.40mm_HandSolder, F.Cu at (57.5, 32.2)
- added R5: 22, 3x6_components:R_0805_2012Metric_Pad1.20x1.40mm_HandSolder, F.Cu at (66.3, 55.2)
- added R6: 10K, 3x6_components:R_0805_2012Metric_Pad1.20x1.40mm_HandSolder, F.Cu at (44.4, 67.6)
- added R7: 720, 3x6_components:R_0805_2012Metric_Pad1.20x1.40mm_HandSolder, F.Cu at (45.0, 38.1)
- added SWR1: SW_Push, 3x6_components:SW_SPST_TL3342, F.Cu at (72.3, 60.3)
- added U2: ATMEGA32U4_QFN44, 3x6_components:TQFP-44_10x10mm_P0.8mm, F.Cu at (53.0, 62.6)
- added USB1: USB_C_HRO-TYPE-C-31-M-12, 3x6_connectors:USB_C-31-M-12, F.Cu at (67.5, 29.0)
- added Y1: 16MHz_Crystal_GND24, 3x6_components:Crystal_SMD_TXC_7M-4Pin_3.2x2.5mm_HandSoldering, F.Cu at (53.4, 52.5)
- D0, D1, D11, D12, D13, D14, D15, D2, D20, D21, D22, D23, D24, D25, D26, D3, D30, D31, D34, D35, D36, D4, D40, D45, D46, D5: footprint kudox_game_footprints:Diode-dual -> 3x6_components:D_THT_7.62_SOD-123_Single_Side
- K0, K1, K11, K12, K13, K14, K15, K2, K20, K21, K22, K23, K24, K25, K26, K3, K31, K34, K35, K36, K4, K5: footprint kudox_game_footprints:MX_socket_optional_100 -> 3x6_kailh_switch:SW_Hotswap_Kailh_1.00u
- K30, K40, K45: footprint kudox_game_footprints:MX_socket_optional_150 -> 3x6_kailh_switch:SW_Hotswap_Kailh_1.50u
- K46: footprint kudox_game_footprints:MX_socket_optional_200 -> 3x6_kailh_switch:SW_Hotswap_Kailh_2.00u
- U1: value ProMicro -> USBLC6-2SC6; footprint kudox_game_footprints:ArduinoProMicro -> 3x6_components:SOT-23-6_Handsoldering; moved to F.Cu
- moved D46 37.4 mm to (147.6, 126.8), turned to 90 degrees
- moved D45 15.7 mm to (149.7, 126.8), turned to 90 degrees
- moved D0 15.4 mm to (53.4, 49.3)
- moved U1 13.4 mm to (67.2, 49.8)
- moved D40 13.2 mm to (58.5, 125.3), turned to 180 degrees
- turned K0 to 180 degrees
- turned K1 to 180 degrees
- turned K11 to 180 degrees
- turned K12 to 180 degrees
- turned K13 to 180 degrees
- turned K14 to 180 degrees
- turned K15 to 180 degrees
- turned K2 to 180 degrees
- turned K20 to 180 degrees
- turned K21 to 180 degrees
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Connections:
- U1 pad 1: rgb_data -> /RAW_D-
- U1 pad 2: Net-(U1-Pad2) -> GND
- U1 pad 3: GND -> /RAW_D+
- U1 pad 4: GND -> /DR+
- U1 pad 5: Net-(U1-Pad5) -> VCC
- U1 pad 6: Net-(U1-Pad6) -> /DR-
Routing:
- net +5V: track 0.00 -> 775.6 mm, vias 0 -> 9
- net VCC: track 245.0 -> 24.0 mm, vias 0 -> 2
- net rgb_data: track 205.3 -> 0.00 mm
- net GND: track 205.5 -> 9.81 mm, vias 0 -> 45
- net RST: track 156.9 -> 0.00 mm
- net col5: track 331.5 -> 196.0 mm, vias 0 -> 7
- net col3: track 235.0 -> 105.7 mm, vias 0 -> 5
- net col6: track 308.2 -> 187.1 mm, vias 0 -> 5
- net col4: track 263.1 -> 146.8 mm, vias 0 -> 6
- net Net-(LED40-Pad2): track 0.00 -> 107.6 mm
- net col1: track 156.4 -> 97.7 mm, vias 0 -> 6
- net col2: track 140.9 -> 92.2 mm, vias 0 -> 5
- net Net-(LED11-Pad2): track 0.00 -> 48.6 mm, vias 0 -> 2
- net row4: track 213.7 -> 169.1 mm, vias 0 -> 1
- net Net-(LED30-Pad2): track 0.00 -> 38.4 mm, vias 0 -> 2
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Other:
- net class Default removed
- board text removed: "DIN"
- board text removed: "GND"
- board text removed: "Mounting Surface"
- board text removed: "VCC"
